File: kicad/TTLSerialOptoisolator.kicad_pcb (KiCad board)
At the start: 2 copper layers, 8 parts, among them P1 CONN_4, P2 CONN_4, U1 817C, U2 817C

Commit message: iterating on board layout
Parts:
- added G***: OSHW-logo_silkscreen-back_2mm, OSHW-logo_silkscreen-back_2mm, F.Cu at (139.1, 74.3)
- moved R3 14.7 mm to (146.7, 66.0), turned to 0 degrees
- moved R4 13.6 mm to (146.7, 68.6), turned to 0 degrees
- moved U2 12.1 mm to (140.3, 67.3)
- moved R1 10.0 mm to (136.5, 71.8), turned to 0 degrees
- moved R2 10.0 mm to (146.7, 74.3), turned to 180 degrees
- moved P1 7.62 mm to (132.7, 69.8)
- moved P2 3.81 mm to (160.7, 69.8)
- moved U1 0.90 mm to (153.0, 73.0)
Routing:
- net N-000003: track 2.54 -> 14.4 mm
- net N-0000010: track 2.54 -> 13.0 mm
- net RXa: track 14.2 -> 23.6 mm
- net 5Vb: track 9.83 -> 17.6 mm
- net TXb: track 12.0 -> 4.86 mm
- net TXa: track 9.83 -> 5.13 mm
- net 5Va: track 16.5 -> 20.0 mm
- net RXb: track 16.4 -> 18.0 mm
Other:
- board outline added: 30.5 x 12.1 mm
- board text added: "5V"
- board text added: "GND"
- board text added: "RX"
- board text added: "TTL Serial Optoisolator"
- board text added: "TX"
- board text added: "github.com/ pepaslabs/ TTLSerialOptoisolator"
- board text added: "v1"

Commit message: changing LED resistor values to 330 ohm.
Parts:
- R1, R4: value 470 -> 330
Changed lines of the file:
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@@
     (links 14)
     (no_connects 0)
-    (area 0 0 0 0)
+    (area 129.3114 63.754 162.306001 76.327)
     (thickness 1.6)
     (drawings 15)
@@
   (page A3)
   (layers
-    (15 F.Cu signal hide)
-    (0 B.Cu signal hide)
+    (15 F.Cu signal)
+    (0 B.Cu signal)
     (16 B.Adhes user)
     (17 F.Adhes user)
@@
   )
   (setup
-    (last_trace_width 0.381)
+    (last_trace_width 0.254)
     (user_trace_width 0.381)
     (user_trace_width 0.508)
@@
       (effects (font (size 0.762 0.762) (thickness 0.1524)))
     )
-    (fp_text value 470 (at 7.112 0) (layer F.SilkS)
+    (fp_text value 330 (at 7.112 0) (layer F.SilkS)
       (effects (font (size 0.762 0.762) (thickness 0.1524)))
     )
@@
       (effects (font (size 0.762 0.762) (thickness 0.1524)))
     )
-    (fp_text value 470 (at 7.112 0) (layer F.SilkS)
+    (fp_text value 330 (at 7.112 0) (layer F.SilkS)
       (effects (font (size 0.762 0.762) (thickness 0.1524)))
     )

Commit message: creating gerbers for board v1.
Parts:
- R2, R3: value 10k -> 4.7k
Other:
- board text added: "Master"
- board text added: "Slave"
Changed lines of the file:
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@@
     (area 129.3114 63.754 162.306001 76.327)
     (thickness 1.6)
-    (drawings 15)
+    (drawings 17)
     (tracks 46)
     (zones 0)
@@
     (19 F.Paste user)
     (20 B.SilkS user)
-    (21 F.SilkS user hide)
+    (21 F.SilkS user)
     (22 B.Mask user)
     (23 F.Mask user)
@@
     (visible_elements 7FFFFFFF)
     (pcbplotparams
-      (layerselection 3178497)
+      (layerselection 284196865)
       (usegerberextensions true)
       (excludeedgelayer true)
@@
       (outputformat 1)
       (mirror false)
-      (drillshape 1)
+      (drillshape 0)
       (scaleselection 1)
-      (outputdirectory ""))
+      (outputdirectory gerbers/))
   )
   (net 0 "")
@@
       (effects (font (size 0.762 0.762) (thickness 0.1524)))
     )
-    (fp_text value 10k (at 7.112 0 180) (layer F.SilkS)
+    (fp_text value 4.7k (at 7.112 0 180) (layer F.SilkS)
       (effects (font (size 0.762 0.762) (thickness 0.1524)))
     )
@@
       (effects (font (size 0.762 0.762) (thickness 0.1524)))
     )
-    (fp_text value 10k (at 7.112 0) (layer F.SilkS)
+    (fp_text value 4.7k (at 7.112 0) (layer F.SilkS)
       (effects (font (size 0.762 0.762) (thickness 0.1524)))
     )
@@
       (xy 0.60452 0.89662)) (layer B.SilkS) (width 0.00254))
   )
+  (gr_text Slave (at 161.29 75.565) (layer B.SilkS)
+    (effects (font (size 0.635 0.635) (thickness 0.127)) (justify left mirror))
+  )
+  (gr_text Master (at 135.255 75.565) (layer B.SilkS)
+    (effects (font (size 0.635 0.635) (thickness 0.127)) (justify left mirror))
+  )
   (gr_text GND (at 159.385 73.025) (layer B.SilkS)
